Commit message: Added Kinect sensor to robot description
Altered the robot description and launcher in order to have a Microsoft Kinect depth sensor in a simulated Gazebo environment.
Tested in Ubuntu 16.04, ROS Kinetic, Gazebo 7.0.0

File: baxter_description/urdf/baxter.urdf.xacro (robot description, xacro)
@@ -1,9 +1,12 @@
 <?xml version="1.0" ?>
 <robot name="baxter" xmlns:xacro="http://www.ros.org/wiki/xacro">
+  <xacro:property name="M_PI" value="3.14159265359" />
   <xacro:arg name="gazebo" default="false"/>
   <xacro:arg name="pedestal" default="true"/>
+  <xacro:arg name="kinect" default="false"/>
   <!-- Baxter Base URDF -->
   <xacro:include filename="$(find baxter_description)/urdf/baxter_base/baxter_base.urdf.xacro">
     <xacro:arg name="gazebo" value="${gazebo}"/>
+    <xacro:arg name="kinect" value="${kinect}"/>
   </xacro:include>
   <!-- Baxter Pedestal -->

File: baxter_description/urdf/baxter_base/baxter_base.gazebo.xacro (robot description, xacro)
@@ -1,4 +1,6 @@
 <?xml version="1.0" ?>
 <robot name="baxter" xmlns:xacro="http://www.ros.org/wiki/xacro">
+  <!-- Whether to include a kinect depth sensor or not -->
+  <xacro:arg name="kinect" default="false"/>
   <!-- ros_control plugin -->
   <gazebo>
@@ -286,4 +288,49 @@
     </sensor>
   </gazebo>
+  <!-- Kinect simulation in gazebo -->
+  <xacro:if value="$(arg kinect)">
+    <gazebo reference="kinect_link">
+      <sensor name="camera" type="depth">
+        <update_rate>30.0</update_rate>
+        <camera>
+          <horizontal_fov>1.047198</horizontal_fov>
+          <image>
+            <width>640</width>
+            <height>480</height>
+            <format>R8G8B8</format>
+          </image>
+          <clip>
+            <near>0.05</near>
+            <far>3</far>
+          </clip>
+        </camera>
+        <plugin name="camera_plugin" filename="libgazebo_ros_openni_kinect.so">
+          <baseline>0.2</baseline>
+          <alwaysOn>true</alwaysOn>
+          <!-- Keep this zero, update_rate in the parent <sensor> tag
+            will control the frame rate. -->
+          <updateRate>0.0</updateRate>
+          <cameraName>camera_ir</cameraName>
+          <imageTopicName>/camera/depth/image_raw</imageTopicName>
+          <cameraInfoTopicName>/camera/depth/camera_info</cameraInfoTopicName>
+          <depthImageTopicName>/camera/depth/image_raw</depthImageTopicName>
+          <depthImageInfoTopicName>/camera/depth/camera_info</depthImageInfoTopicName>
+          <pointCloudTopicName>/camera/depth/points</pointCloudTopicName>
+          <frameName>kinect_depth_frame</frameName>
+          <pointCloudCutoff>0.05</pointCloudCutoff>
+          <distortionK1>0</distortionK1>
+          <distortionK2>0</distortionK2>
+          <distortionK3>0</distortionK3>
+          <distortionT1>0</distortionT1>
+          <distortionT2>0</distortionT2>
+          <CxPrime>0</CxPrime>
+          <Cx>0</Cx>
+          <Cy>0</Cy>
+          <focalLength>0</focalLength>
+          <hackBaseline>0</hackBaseline>
+        </plugin>
+      </sensor>
+    </gazebo>
+  </xacro:if>
   <!-- Transmissions -->
   <!-- Right Arm -->

File: baxter_description/urdf/baxter_base/baxter_base.urdf.xacro (robot description, xacro)
@@ -2,4 +2,5 @@
 <robot name="baxter" xmlns:xacro="http://www.ros.org/wiki/xacro">
   <xacro:arg name="gazebo" default="false"/>
+  <xacro:arg name="kinect" default="false"/>
   <xacro:if value="$(arg gazebo)">
     <!-- Gazebo Tags -->
@@ -875,4 +876,36 @@
     </inertial>
   </link>
+  <!-- Kinect Depth Sensor -->
+  <xacro:if value="$(arg kinect)">
+    <joint name="kinect_joint" type="fixed">
+      <origin rpy="0 0 0" xyz="0.3 0 0"/>
+      <parent link="base"/>
+      <child link="kinect_link"/>
+    </joint>
+    <link name="kinect_link">
+      <collision name="collision">
+        <origin rpy="0 0 0"
+                xyz="0 0 0"/>
+        <geometry>
+          <box size="0.073000 0.276000 0.072000"/>
+        </geometry>
+      </collision>
+      <visual>
+        <origin rpy="0 0 0"
+                xyz="0 0 0"/>
+        <geometry>
+          <mesh filename="package://baxter_description/meshes/kinect/meshes/kinect.dae"/>
+        </geometry>
+      </visual>
+    </link>
+    <joint name="kinect_depth_joint" type="fixed">
+      <origin rpy="${-M_PI/2} 0 ${-M_PI/2}"
+              xyz="0 0 0"/>
+      <parent link="kinect_link" />
+      <child link="kinect_depth_frame" />
+    </joint>
+    <link name="kinect_depth_frame">
+    </link>
+  </xacro:if>
   <joint name="left_torso_arm_mount" type="fixed">
     <origin rpy="0 0 0.7854" xyz="0.024645 0.219645 0.118588"/>
